File: Board_eagle/ATTint_SOMO-4D.sch (EAGLE design)
At the start: 18 parts, among them U1 SOMO-14D, U2 MAX1555, X2 STEREOJACK, X3 USB-SMD-NS

Commit message: Code cleaning
Parts:
- added R1: 1K, spark-fun:RESISTOR
Connections:
- net CLOCK: now also U$6.PB1(MISO); no longer U$6.PB0(MOSI)
- net DATA: now also U$6.PB2(SCK/ADC1); no longer U$6.PB1(MISO)
- net RESET: now also U$6.PB0(MOSI); no longer U$6.PB2(SCK/ADC1)
- net SWITCH: now also R1.2
- net VCC: now also R1.1
Changed lines of the file:
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@@
 <part name="AUDIO1" library="SparkFun" deviceset="M02" device="LOCK_LONGPADS" value="3.3V"/>
 <part name="SWITCH1" library="SparkFun" deviceset="SWITCH-MOMENTARY-2" device="SMD"/>
+<part name="R1" library="spark-fun" deviceset="RESISTOR" device="" value="1K"/>
+<part name="P+4" library="supply1" deviceset="VCC" device=""/>
 </parts>
 <sheets>
@@
 <instance part="AUDIO1" gate="G$1" x="73.66" y="73.66" rot="R180"/>
 <instance part="SWITCH1" gate="G$1" x="83.82" y="-25.4" rot="R180"/>
+<instance part="R1" gate="G$1" x="73.66" y="0" rot="R270"/>
+<instance part="P+4" gate="VCC" x="73.66" y="12.7"/>
 </instances>
 <busses>
@@
 <wire x1="48.26" y1="50.8" x2="22.86" y2="50.8" width="0.1524" layer="91"/>
 <junction x="22.86" y="50.8"/>
+</segment>
+<segment>
+<pinref part="R1" gate="G$1" pin="1"/>
+<pinref part="P+4" gate="VCC" pin="VCC"/>
+<wire x1="73.66" y1="5.08" x2="73.66" y2="10.16" width="0.1524" layer="91"/>
 </segment>
 </net>
@@
 <net name="CLOCK" class="0">
 <segment>
-<wire x1="22.86" y1="-20.32" x2="38.1" y2="-20.32" width="0.1524" layer="91"/>
-<label x="38.1" y="-20.32" size="1.778" layer="95"/>
-<pinref part="U$6" gate="G$1" pin="PB0(MOSI)"/>
-</segment>
-<segment>
 <pinref part="U1" gate="SOMO-14D" pin="CLK"/>
 <wire x1="-7.62" y1="60.96" x2="-15.24" y2="60.96" width="0.1524" layer="91"/>
 <label x="-22.86" y="60.96" size="1.778" layer="95"/>
 <junction x="-7.62" y="60.96"/>
+</segment>
+<segment>
+<pinref part="U$6" gate="G$1" pin="PB1(MISO)"/>
+<wire x1="22.86" y1="-22.86" x2="38.1" y2="-22.86" width="0.1524" layer="91"/>
+<label x="38.1" y="-22.86" size="1.778" layer="95"/>
 </segment>
 </net>
@@
 <net name="DATA" class="0">
 <segment>
-<pinref part="U$6" gate="G$1" pin="PB1(MISO)"/>
-<wire x1="22.86" y1="-22.86" x2="38.1" y2="-22.86" width="0.1524" layer="91"/>
-<label x="38.1" y="-22.86" size="1.778" layer="95"/>
-</segment>
-<segment>
 <pinref part="U1" gate="SOMO-14D" pin="DATA"/>
 <wire x1="-7.62" y1="58.42" x2="-15.24" y2="58.42" width="0.1524" layer="91"/>
 <label x="-22.86" y="58.42" size="1.778" layer="95"/>
 <junction x="-7.62" y="58.42"/>
+</segment>
+<segment>
+<pinref part="U$6" gate="G$1" pin="PB2(SCK/ADC1)"/>
+<wire x1="22.86" y1="-25.4" x2="38.1" y2="-25.4" width="0.1524" layer="91"/>
+<label x="38.1" y="-25.4" size="1.778" layer="95"/>
 </segment>
 </net>
@@
 <net name="SWITCH" class="0">
 <segment>
-<wire x1="81.28" y1="-10.16" x2="76.2" y2="-10.16" width="0.1524" layer="91"/>
-<label x="66.04" y="-10.16" size="1.778" layer="95"/>
+<wire x1="81.28" y1="-10.16" x2="73.66" y2="-10.16" width="0.1524" layer="91"/>
+<label x="53.34" y="-10.16" size="1.778" layer="95"/>
 <pinref part="SWITCH" gate="G$1" pin="1"/>
 <junction x="81.28" y="-10.16"/>
+<pinref part="R1" gate="G$1" pin="2"/>
+<wire x1="73.66" y1="-10.16" x2="63.5" y2="-10.16" width="0.1524" layer="91"/>
+<wire x1="73.66" y1="-5.08" x2="73.66" y2="-10.16" width="0.1524" layer="91"/>
+<junction x="73.66" y="-10.16"/>
 </segment>
 <segment>
@@
 </segment>
 <segment>
-<pinref part="U$6" gate="G$1" pin="PB2(SCK/ADC1)"/>
-<wire x1="22.86" y1="-25.4" x2="38.1" y2="-25.4" width="0.1524" layer="91"/>
-<label x="38.1" y="-25.4" size="1.778" layer="95"/>
-</segment>
-</net>
+<wire x1="22.86" y1="-20.32" x2="38.1" y2="-20.32" width="0.1524" layer="91"/>
+<label x="38.1" y="-20.32" size="1.778" layer="95"/>
+<pinref part="U$6" gate="G$1" pin="PB0(MOSI)"/>
+</segment>
+</net>

Commit message: optimised sleeping consumption
Parts:
- removed X2: STEREOJACK, adafruit:STEREOJACK
- added R2: 1K, spark-fun:RESISTOR
- added SENSOR_A: 3.3V, charles:M02LOCK_LONGPADS
- added U3: (no value), SparkFun:AUDIO-JACKSMD2
- renumbered SENSOR to SENSOR_B
Connections:
- net AUDIO_A: now also U3.SLEEVE; no longer X2.1
- net AUDIO_B: now also U3.LEFT, U3.RIGHT; no longer X2.2, X2.3, X2.4, X2.5
- net GND: now also R2.2
- net NRESET: now also R2.1, SENSOR_A.2
- net VCC: now also SENSOR_A.1
Changed lines of the file:
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@@
 <part name="P+1" library="supply1" deviceset="VCC" device=""/>
 <part name="GND1" library="spark-fun" deviceset="GND" device=""/>
-<part name="X2" library="adafruit" deviceset="STEREOJACK" device=""/>
 <part name="GND9" library="supply1" deviceset="GND" device=""/>
 <part name="GND8" library="supply1" deviceset="GND" device=""/>
 <part name="U$6" library="SparkFun" deviceset="ATTINY13" device="DIP"/>
 <part name="U1" library="SpaElectronics" deviceset="SOMO-14D" device=""/>
-<part name="SENSOR" library="charles" deviceset="M02" device="LOCK_LONGPADS" value="3.3V"/>
+<part name="SENSOR_B" library="charles" deviceset="M02" device="LOCK_LONGPADS" value="3.3V"/>
 <part name="P+2" library="supply1" deviceset="VCC" device=""/>
 <part name="GND3" library="spark-fun" deviceset="GND" device=""/>
@@
 <part name="R1" library="spark-fun" deviceset="RESISTOR" device="" value="1K"/>
 <part name="P+4" library="supply1" deviceset="VCC" device=""/>
+<part name="U3" library="SparkFun" deviceset="AUDIO-JACK" device="SMD2"/>
+<part name="R2" library="spark-fun" deviceset="RESISTOR" device="" value="1K"/>
+<part name="GND6" library="supply1" deviceset="GND" device=""/>
+<part name="SENSOR_A" library="charles" deviceset="M02" device="LOCK_LONGPADS" value="3.3V"/>
 </parts>
 <sheets>
@@
 <instance part="P+1" gate="VCC" x="-10.16" y="-10.16"/>
 <instance part="GND1" gate="1" x="-10.16" y="-40.64"/>
-<instance part="X2" gate="1" x="99.06" y="45.72" rot="MR180"/>
 <instance part="GND9" gate="1" x="96.52" y="-15.24"/>
 <instance part="GND8" gate="1" x="86.36" y="5.08"/>
 <instance part="U$6" gate="G$1" x="10.16" y="-27.94"/>
 <instance part="U1" gate="SOMO-14D" x="7.62" y="58.42"/>
-<instance part="SENSOR" gate="G$1" x="101.6" y="25.4" rot="R180"/>
+<instance part="SENSOR_B" gate="G$1" x="101.6" y="25.4" rot="R180"/>
 <instance part="P+2" gate="VCC" x="48.26" y="73.66"/>
 <instance part="GND3" gate="1" x="25.4" y="43.18"/>
@@
 <instance part="R1" gate="G$1" x="73.66" y="0" rot="R270"/>
 <instance part="P+4" gate="VCC" x="73.66" y="12.7"/>
+<instance part="U3" gate="G$1" x="91.44" y="40.64" rot="R180"/>
+<instance part="R2" gate="G$1" x="33.02" y="15.24" rot="R270"/>
+<instance part="GND6" gate="1" x="33.02" y="5.08"/>
+<instance part="SENSOR_A" gate="G$1" x="48.26" y="25.4" rot="R180"/>
 </instances>
 <busses>
@@
 <wire x1="93.98" y1="25.4" x2="76.2" y2="25.4" width="0.1524" layer="91"/>
 <label x="71.12" y="25.4" size="1.778" layer="95"/>
-<pinref part="SENSOR" gate="G$1" pin="1"/>
+<pinref part="SENSOR_B" gate="G$1" pin="1"/>
 </segment>
 <segment>
@@
 <pinref part="P+4" gate="VCC" pin="VCC"/>
 <wire x1="73.66" y1="5.08" x2="73.66" y2="10.16" width="0.1524" layer="91"/>
+</segment>
+<segment>
+<wire x1="40.64" y1="25.4" x2="22.86" y2="25.4" width="0.1524" layer="91"/>
+<pinref part="SENSOR_A" gate="G$1" pin="1"/>
+<label x="17.78" y="25.4" size="1.778" layer="95"/>
 </segment>
 </net>
@@
 <pinref part="SWITCH1" gate="G$1" pin="1"/>
 </segment>
+<segment>
+<pinref part="R2" gate="G$1" pin="2"/>
+<pinref part="GND6" gate="1" pin="GND"/>
+<wire x1="33.02" y1="10.16" x2="33.02" y2="7.62" width="0.1524" layer="91"/>
+</segment>
 </net>
 <net name="CLOCK" class="0">
@@
 <label x="71.12" y="22.86" size="1.778" layer="95"/>
 <pinref part="R7" gate="G$1" pin="1"/>
-<pinref part="SENSOR" gate="G$1" pin="2"/>
+<pinref part="SENSOR_B" gate="G$1" pin="2"/>
 </segment>
 <segment>
@@
 </segment>
 <segment>
-<pinref part="X2" gate="1" pin="1"/>
-<wire x1="71.12" y1="53.34" x2="86.36" y2="53.34" width="0.1524" layer="91"/>
-<label x="66.04" y="53.34" size="1.778" layer="95"/>
+<wire x1="81.28" y1="38.1" x2="86.36" y2="38.1" width="0.1524" layer="91"/>
+<label x="66.04" y="38.1" size="1.778" layer="95"/>
+<pinref part="U3" gate="G$1" pin="SLEEVE"/>
+<junction x="86.36" y="38.1"/>
 </segment>
 </net>
@@
 </segment>
 <segment>
-<wire x1="83.82" y1="43.18" x2="76.2" y2="43.18" width="0.1524" layer="91"/>
 <label x="66.04" y="43.18" size="1.778" layer="95"/>
-<pinref part="X2" gate="1" pin="2"/>
-<wire x1="86.36" y1="50.8" x2="83.82" y2="50.8" width="0.1524" layer="91"/>
-<wire x1="83.82" y1="50.8" x2="83.82" y2="48.26" width="0.1524" layer="91"/>
-<pinref part="X2" gate="1" pin="5"/>
-<wire x1="83.82" y1="48.26" x2="83.82" y2="45.72" width="0.1524" layer="91"/>
-<wire x1="83.82" y1="45.72" x2="83.82" y2="43.18" width="0.1524" layer="91"/>
-<wire x1="83.82" y1="43.18" x2="86.36" y2="43.18" width="0.1524" layer="91"/>
-<pinref part="X2" gate="1" pin="4"/>
-<wire x1="86.36" y1="45.72" x2="83.82" y2="45.72" width="0.1524" layer="91"/>
-<junction x="83.82" y="45.72"/>
-<pinref part="X2" gate="1" pin="3"/>
-<wire x1="86.36" y1="48.26" x2="83.82" y2="48.26" width="0.1524" layer="91"/>
-<junction x="83.82" y="48.26"/>
-<junction x="83.82" y="43.18"/>
+<pinref part="U3" gate="G$1" pin="LEFT"/>
+<wire x1="81.28" y1="43.18" x2="76.2" y2="43.18" width="0.1524" layer="91"/>
+<wire x1="86.36" y1="43.18" x2="81.28" y2="43.18" width="0.1524" layer="91"/>
+<wire x1="81.28" y1="43.18" x2="81.28" y2="40.64" width="0.1524" layer="91"/>
+<pinref part="U3" gate="G$1" pin="RIGHT"/>
+<wire x1="81.28" y1="40.64" x2="86.36" y2="40.64" width="0.1524" layer="91"/>
+<junction x="86.36" y="43.18"/>
+<junction x="86.36" y="40.64"/>
 </segment>
 </net>
@@
 <pinref part="SWITCH1" gate="G$1" pin="2"/>
 </segment>
-</net>
+<segment>
+<wire x1="33.02" y1="22.86" x2="33.02" y2="20.32" width="0.1524" layer="91"/>
+<wire x1="33.02" y1="22.86" x2="22.86" y2="22.86" width="0.1524" layer="91"/>
+<wire x1="40.64" y1="22.86" x2="33.02" y2="22.86" width="0.1524" layer="91"/>
+<junction x="33.02" y="22.86"/>
+<pinref part="R2" gate="G$1" pin="1"/>
+<pinref part="SENSOR_A" gate="G$1" pin="2"/>
+<label x="17.78" y="22.86" size="1.778" layer="95"/>
+</segment>
+</net>
